Commit message: refactor rbfiqus_agrimate files, xacro and urdf

File: robots/rbfiqus_agrimate/rbfiqus_agrimate.urdf.xacro (robot description, xacro)
@@ -1,8 +1,8 @@
 <?xml version="1.0" ?>
 <robot
-  name="rbfiqus"
+  name="rbfiqus_agrimate"
   xmlns:xacro="http://wiki.ros.org/xacro">
   <xacro:include
-    filename="$(find robotnik_description)/urdf/bases/rbfiqus/rbfiqus_agrimate_base.urdf.xacro" />
+    filename="$(find robotnik_description)/urdf/bases/rbfiqus_agrimate/rbfiqus_agrimate_base.urdf.xacro" />
   <xacro:include
     filename="$(find robotnik_sensors)/urdf/all_sensors.urdf.xacro" />
@@ -22,6 +22,6 @@
     name="ur_type"
     default="ur5e" />
-  <!-- RB-FIQUS -->
-  <xacro:rbfiqus
+  <!-- RB-FIQUS AGRIMATE -->
+  <xacro:rbfiqus_agrimate
     prefix="$(arg prefix)"
     gazebo_ignition="$(arg gazebo_ignition)"
@@ -38,5 +38,5 @@
   </xacro:sensor_vectornav>
   <!-- ARMS -->
-  <xacro:arm_ur
+  <!--<xacro:arm_ur
     ur_type="$(arg ur_type)"
     frame_prefix="$(arg prefix)arm1_"
@@ -55,5 +55,5 @@
       xyz="0.005 -0.7 0.542"
       rpy="0 0 0" />
-  </xacro:arm_ur >
+  </xacro:arm_ur > -->
     <!-- LASERS -->
   <!--xacro:sensor_robosense_bpearl
@@ -105,3 +105,14 @@
       rpy="${pi} ${-1.52*pi} 0" />
   </xacro:sensor_robosense_bpearl>
+  <!-- GPS -->
+  <xacro:sensor_ublox_with_mast
+    frame_prefix="$(arg prefix)gps_"
+    parent="$(arg prefix)base_link"
+    node_namespace="$(arg namespace)"
+    node_name="gps"
+    gazebo_ignition="$(arg gazebo_ignition)">
+    <origin
+      xyz="0.0 0.0 2.0"
+      rpy="0 0 0" />
+  </xacro:sensor_ublox_with_mast>
 </robot>

File: urdf/bases/rbfiqus_agrimate/rbfiqus_agrimate_base.urdf.xacro (robot description, xacro)
@@ -1,5 +1,5 @@
 <?xml version="1.0" ?>
 <robot
-  name="rbfiqus_base"
+  name="rbfiqus_agrimate_base"
   xmlns:xacro="http://www.ros.org/wiki/xacro">
   <xacro:include
@@ -10,17 +10,26 @@
     filename="$(find robotnik_description)/urdf/wheels/steering_wheel/wheel_rbfiqus_agrimate_back.urdf.xacro" />
   <xacro:include
-    filename="$(find robotnik_description)/simulators/gazebo_ignition/rbfiqus/rbfiqus_control.urdf.xacro" />
+    filename="$(find robotnik_description)/simulators/gazebo_ignition/rbfiqus_agrimate/rbfiqus_agrimate_control.urdf.xacro" />
   <!-- WHEELS PROPERTIES -->
   <xacro:property
-    name="wheel_offset_x"
+    name="front_wheel_offset_x"
     value="0.750" />
   <xacro:property
-    name="wheel_offset_y"
+    name="front_wheel_offset_y"
     value="0.9211" />
   <xacro:property
-    name="wheel_offset_z"
+    name="front_wheel_offset_z"
     value="0.15" />
+  <xacro:property
+    name="back_wheel_offset_x"
+    value="-0.822" />
+  <xacro:property
+    name="back_wheel_offset_y"
+    value="0.7779" />
+  <xacro:property
+    name="back_wheel_offset_z"
+    value="0.13619" />
   <xacro:macro
-    name="rbfiqus"
+    name="rbfiqus_agrimate"
     params="
       prefix:=robot_
@@ -40,5 +49,5 @@
       hq="${hq}">
       <origin
-        xyz="${wheel_offset_x} -${wheel_offset_y} ${wheel_offset_z}"
+        xyz="${front_wheel_offset_x} -${front_wheel_offset_y} ${front_wheel_offset_z}"
         rpy="0 0 0" />
     </xacro:steering_wheel_rbfiqus_agrimate>
@@ -49,5 +58,5 @@
       hq="${hq}">
       <origin
-        xyz="${wheel_offset_x} ${wheel_offset_y} ${wheel_offset_z}"
+        xyz="${front_wheel_offset_x} ${front_wheel_offset_y} ${front_wheel_offset_z}"
         rpy="0 0 0" />
     </xacro:steering_wheel_rbfiqus_agrimate>
@@ -59,5 +68,5 @@
       left="true">
       <origin
-        xyz="-0.822 0.7779 0.13619"
+        xyz="${back_wheel_offset_x} ${back_wheel_offset_y} ${back_wheel_offset_z}"
         rpy="0 0 0" />
     </xacro:wheel_rbfiqus_agrimate_back>
@@ -69,9 +78,9 @@
       left="false">
       <origin
-        xyz="-0.822 -0.7779 0.13619"
+        xyz="${back_wheel_offset_x} -${back_wheel_offset_y} ${back_wheel_offset_z}"
         rpy="0 0 0" />
     </xacro:wheel_rbfiqus_agrimate_back>
     <xacro:if value="$(arg gazebo_ignition)">
-      <xacro:rbfiqus_gz_ignition_control
+      <xacro:rbfiqus_agrimate_gz_ignition_control
         namespace="${namespace}"
         prefix="${prefix}" />

File: urdf/bodies/rbfiqus/rbfiqus_agrimate_body.urdf.xacro (robot description, xacro)
@@ -54,14 +54,25 @@
             </inertial>
         </link>
-    <!-- DOCKING CONTACT -->
-    <link name="${prefix}base_docking_contact" />
+    <!-- Front axle control frame used by docking/navigation tests. -->
+    <link name="${prefix}base_docking_control" />
     <joint
       name="${prefix}base_docking_joint"
       type="fixed">
       <origin
-        xyz="0.6405 0 0.10264"
+        xyz="0.750 0 0"
         rpy="0 0 0" />
-      <parent link="${prefix}chassis_link" />
-      <child link="${prefix}base_docking_contact" />
+      <parent link="${prefix}base_link" />
+      <child link="${prefix}base_docking_control" />
+    </joint>
+    <!-- Rear axle frame for comparing base/front/rear axle trajectories. -->
+    <link name="${prefix}base_rear_axle" />
+    <joint
+      name="${prefix}base_rear_axle_joint"
+      type="fixed">
+      <origin
+        xyz="-0.822 0 0"
+        rpy="0 0 0" />
+      <parent link="${prefix}base_link" />
+      <child link="${prefix}base_rear_axle" />
     </joint>
   </xacro:macro>
